File: Hardware/keyboard_mouse_board/kb_mouse.kicad_sch (KiCad schematic)
At the start: 25 parts, among them J1 Conn_01x40, J2 Conn_01x02, J3 AVR-ISP-6, U1 74HC74, U2 ATmega328P-P, U3 DS1307+, U4 74HC245, U5 74HC00, Y1 32,768kHz

Commit message: RDY latch fix
Parts:
- removed J2: Conn_01x02, Connector_PinHeader_2.54mm:PinHeader_1x02_P2.54mm_Vertical, symbol Connector_Generic:Conn_01x02
- added C5: 100n, Capacitor_THT:C_Disc_D5.0mm_W2.5mm_P5.00mm, symbol Device:C
- added JP1: CLK_RESET, Connector_PinHeader_2.54mm:PinHeader_1x02_P2.54mm_Vertical, symbol Jumper:Jumper_2_Bridged
- J3: footprint Connector_IDC:IDC-Header_2x03_P2.54mm_Vertical -> Connector_IDC:IDC-Header_2x03_P2.54mm_Horizontal
- RDY1: renamed from D1; footprint LED_THT:LED_D5.0mm -> LED_THT:LED_D3.0mm
- Y1: footprint Crystal:Crystal_C38-LF_D3.0mm_L8.0mm_Horizontal_1EP_style2 -> Crystal:Crystal_DS15_D1.5mm_L5.0mm_Horizontal_1EP_style2
Connections:
- net +5V: now also U1.10 (~{S}), U1.13 (~{R}), C5.1
- net GND: now also U1.11 (C), U1.12 (D), U5.12, U5.13, C5.2
- net at BT1.1 (+): now also JP1.2 (B); no longer U3.3 (VBAT)
- new net: JP1.1 (A), U3.3 (VBAT)
- no-connect marks 6 -> 11
Other:
- note removed: "Jumper to use clock stretching for this board"
- moved on the sheet: R1, R8, RDY1, U1A, U1B, U5D
