File: Hardware/ram_board_AS6/ram_board.kicad_pcb (KiCad board)
At the start: 2 copper layers, 80.8 x 60.1 mm, 16 parts, among them J1 Conn_01x40, U1 74HC00, U2 74HC04, U4 74HC02, U5 74HC273, U6 AS6C4008-55PCN

Commit message: WRITE signal now ative when writing to memmory window
Parts:
- added OSHW2: OSHW-Logo2_7.3x6mm_SilkScreen, Symbol:OSHW-Logo2_7.3x6mm_SilkScreen, B.Cu at (160.0, 84.5)
- moved C6 46.1 mm to (161.3, 124.7)
- moved U6 39.0 mm to (181.6, 121.9), turned to 180 degrees
- moved OSHW1 35.6 mm to (118.1, 84.5)
- moved C4 6.72 mm to (142.2, 108.0), turned to 180 degrees
- moved C7 0.11 mm to (147.5, 104.0)
- moved U4 0.11 mm to (152.5, 93.1)
- moved U5 0.11 mm to (137.2, 118.7)
- renumbered OSHW to OSHW1
Connections:
- U1 pad 6: /~{WE} -> Net-(U1-Pad6)
- U2 pad 5: GND -> Net-(U2-Pad5)
- U2 pad 6: unconnected-(U2-Pad6) -> /~{WE}
- U4 pad 4: unconnected-(U4-Pad4) -> Net-(U2-Pad5)
- U4 pad 5: GND -> /~{OE}
- U4 pad 6: GND -> Net-(U1-Pad6)
Routing:
- net GND: track 86.3 -> 556.3 mm, vias 0 -> 7
- net +5V: track 24.5 -> 364.7 mm, vias 0 -> 4
- net /~{CE}: track 113.7 -> 44.4 mm
- net D6: track 44.5 -> 106.1 mm, vias 0 -> 2
- net D3: track 49.6 -> 111.1 mm, vias 1 -> 0
- net D2: track 52.1 -> 112.9 mm, vias 1 -> 0
- net D0: track 65.5 -> 123.8 mm
- net D5: track 39.8 -> 97.4 mm, vias 0 -> 1
- net D1: track 64.7 -> 120.0 mm
- net A8: track 74.3 -> 24.4 mm
- net D7: track 50.8 -> 100.5 mm, vias 1 -> 0
- net D4: track 55.5 -> 103.7 mm, vias 0 -> 1
- net /RA15: track 66.4 -> 21.8 mm
- net Net-(U1-Pad6): track 0.00 -> 42.4 mm, vias 0 -> 1
- net Net-(U2-Pad5): track 0.00 -> 38.1 mm, vias 0 -> 1
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Other:
- board text added: "AS6 RAM BOARD ${VERSION}"
- board text removed: "RAM BOARD ${VERSION}"
